File: Interface_IAI.kicad_pcb (KiCad board)
At the start: 2 copper layers, 79.3 x 141 mm, 55 parts, among them J1 +24V, J2 Screw_Terminal_01x15, J3 SCON_FEEDBACK, J4 SCON_PULSE, J5 Screw_Terminal_01x14, J6 ADWin CO4-T, U1 AM26LS31, U2 AM26LS32, U3 TBD62783APG, U4 TSR1-2450E

Commit message: Update doc. Change PCB (RSTR, REND, *EMGS)
Connections:
- net /DIO_IN0 renamed /DIO_REN
- net /DIO_IN1 renamed /DIO_EMGS
- net /DIO_OUT0 renamed /RSTR
- net /DIO_OUT1 renamed /DIO_OUT
- net /SCON_IN0 renamed /SCON_RSTR
- net /SCON_IN1 renamed /SCON_IN
- net /SCON_OUT0 renamed /SCON_REN
- net /SCON_OUT1 renamed /SCON_EMGS
Other:
- board text added: "*ALM"
- board text added: "*EMGS"
- board text added: "DIO_OUT"
- board text added: "REN"
- board text added: "REND"
- board text added: "RSTR"
- board text added: "SCON_IN"
- board text removed: "ALM"
- board text removed: "IN0"
- board text removed: "IN1"
- board text removed: "OUT0"
- board text removed: "OUT1"
