File: Interface_IAI.kicad_sch (KiCad schematic)
At the start: 20 parts, among them J1 ADWIN_DIO32, J2 ALIM_5V, J3 SCON_PULSE, J4 SCON_FEEDBACK, J5 ADWIN_CO4T, U1 AM26LS31CN, U2 AM26LS32ACN

Commit message: Update board
Parts:
- removed C2: 10uF, Capacitor_THT:C_Disc_D5.0mm_W2.5mm_P5.00mm, symbol iface:C
- removed J1: ADWIN_DIO32, TerminalBlock_Phoenix:TerminalBlock_Phoenix_MKDS-1,5-3-5.08_1x03_P5.08mm_Horizontal, symbol iface:Conn_R_1x03
- removed J2: ALIM_5V, TerminalBlock_Phoenix:TerminalBlock_Phoenix_MKDS-1,5-2-5.08_1x02_P5.08mm_Horizontal, symbol iface:Conn_R_1x02
- removed J3: SCON_PULSE, TerminalBlock_Phoenix:TerminalBlock_Phoenix_MKDS-1,5-4-5.08_1x04_P5.08mm_Horizontal, symbol iface:Conn_L_1x04
- removed J4: SCON_FEEDBACK, TerminalBlock_Phoenix:TerminalBlock_Phoenix_MKDS-1,5-7-5.08_1x07_P5.08mm_Horizontal, symbol iface:Conn_R_1x07
- removed J5: ADWIN_CO4T, TerminalBlock_Phoenix:TerminalBlock_Phoenix_MKDS-1,5-4-5.08_1x04_P5.08mm_Horizontal, symbol iface:Conn_L_1x04
- removed U1: AM26LS31CN, Package_DIP:DIP-16_W7.62mm_Socket, symbol iface:AM26C31
- removed U2: AM26LS32ACN, Package_DIP:DIP-16_W7.62mm_Socket, symbol iface:AM26C32
- added C4: 10uF, Capacitor_THT:C_Disc_D5.0mm_W2.5mm_P5.00mm, symbol Device:C
- added C5: 10uF 50V, Capacitor_THT:C_Disc_D5.0mm_W2.5mm_P5.00mm, symbol Device:C
- added C6: 100nF, Capacitor_THT:C_Disc_D5.0mm_W2.5mm_P5.00mm, symbol Device:C
- added D1: 1N5819, Diode_THT:D_DO-41_SOD81_P10.16mm_Horizontal, symbol Device:D_Schottky
- added H1, H2, H3, H4: MountingHole, MountingHole:MountingHole_2.2mm_M2, symbol Mechanical:MountingHole
- added J1: +24V, TerminalBlock_Phoenix:TerminalBlock_Phoenix_MKDS-1,5-2-5.08_1x02_P5.08mm_Horizontal, symbol Connector:Screw_Terminal_01x02
- added J2: ADWIN_DIO32, TerminalBlock_Phoenix:TerminalBlock_Phoenix_MKDS-1,5-11-5.08_1x11_P5.08mm_Horizontal, symbol Connector:Screw_Terminal_01x11
- added J3: SCON_FEEDBACK, TerminalBlock_Phoenix:TerminalBlock_Phoenix_MKDS-1,5-7-5.08_1x07_P5.08mm_Horizontal, symbol Connector:Screw_Terminal_01x07
- added J4: SCON_PULSE, TerminalBlock_Phoenix:TerminalBlock_Phoenix_MKDS-1,5-4-5.08_1x04_P5.08mm_Horizontal, symbol Connector:Screw_Terminal_01x04
- added J5: SCON_PIO, TerminalBlock_Phoenix:TerminalBlock_Phoenix_MKDS-1,5-10-5.08_1x10_P5.08mm_Horizontal, symbol Connector:Screw_Terminal_01x10
- added J6: ADWin CO4-T, TerminalBlock_Phoenix:TerminalBlock_Phoenix_MKDS-1,5-4-5.08_1x04_P5.08mm_Horizontal, symbol Connector:Screw_Terminal_01x04
- added R11, R12, R13, R14, R15, R16, R17, R18: 10k, Resistor_THT:R_Axial_DIN0207_L6.3mm_D2.5mm_P7.62mm_Horizontal, symbol Device:R
- added R19, R20, R21, R22: 2.2k, Resistor_THT:R_Axial_DIN0207_L6.3mm_D2.5mm_P7.62mm_Horizontal, symbol Device:R
- added U1: AM26LS31, Package_DIP:DIP-16_W7.62mm_Socket, symbol Interface:AM26LS31CD
- added U2: AM26LS32, Package_DIP:DIP-16_W7.62mm_Socket, symbol Interface:AM26LV32xD
- added U3: TBD62783APG, Package_DIP:DIP-18_W7.62mm_Socket, symbol Transistor_Array:TBD62783A
- added U4: TSR1-2450E, Converter_DCDC:Converter_DCDC_TRACO_TSR-1_THT, symbol Converter_DCDC:TSR1-2450E
- C1, C3: symbol iface:C -> Device:C
- R1, R10, R2, R3, R4, R5, R6, R7, R8, R9: symbol iface:R -> Device:R
Connections:
- net +5V: now also C4.1, U1.16 (VDD), U2.14 (4A), U2.16 (VDD), U4.3 (Vout)
- net A_RX: now also U2.3 (1Y)
- net B_RX: now also U2.5 (2Y)
- net CNT_A: now also J6.3 (Pin_3)
- net CNT_B: now also J6.2 (Pin_2)
- net CNT_Z: now also J6.1 (Pin_1)
- net DIO_PULSE: now also J2.11 (Pin_11)
- net DIO_SIGN: now also J2.10 (Pin_10)
- net FB_A_N: now also J3.1 (Pin_1), U2.1 (1B)
- net FB_A_P: now also J3.2 (Pin_2), U2.2 (1A)
- net FB_B_N: now also J3.4 (Pin_4), U2.7 (2B)
- net FB_B_P: now also J3.3 (Pin_3), U2.6 (2A)
- net FB_Z_N: now also J3.5 (Pin_5), U2.9 (3B)
- net FB_Z_P: now also J3.6 (Pin_6), U2.10 (3A)
- net GND: now also C4.2, C5.2, C6.2, J1.2 (Pin_2), J2.1 (Pin_1), J3.7 (Pin_7), J5.2 (Pin_2), J6.4 (Pin_4), R11.2, R12.2, R13.2, R14.2, R19.2, R20.2, R21.2, R22.2, U1.12 (~{G}), U1.15 (4A), U1.4 (G), U1.8 (GND), U1.9 (3A), U2.12 (~{G}), U2.15 (4B), U2.4 (G), U2.8 (GND), U3.10 (GND), U3.5 (I5), U3.6 (I6), U3.7 (I7), U3.8 (I8), U4.2 (GND)
- net PULSE_N: now also J4.2 (Pin_2), U1.3 (1Z)
- net PULSE_P: now also J4.1 (Pin_1), U1.2 (1Y)
- net PULSE_TTL: now also U1.1 (1A)
- net SIGN_N: now also J4.3 (Pin_3), U1.5 (2Z)
- net SIGN_P: now also J4.4 (Pin_4), U1.6 (2Y)
- net SIGN_TTL: now also U1.7 (2A)
- net Z_RX: now also U2.11 (3Y)
- new net +24V: C6.1, D1.2 (A), J1.1 (Pin_1), J5.1 (Pin_1), U3.9 (VCC)
- new net DIO_ALM: J2.2 (Pin_2), R18.2, R22.1
- new net DIO_CSTP: J2.9 (Pin_9), R14.1, U3.4 (I4)
- new net DIO_HEND: J2.3 (Pin_3), R17.2, R21.1
- new net DIO_HOME: J2.8 (Pin_8), R13.1, U3.3 (I3)
- new net DIO_INP: J2.4 (Pin_4), R16.2, R20.1
- new net DIO_RES: J2.7 (Pin_7), R12.1, U3.2 (I2)
- new net DIO_SON: J2.6 (Pin_6), R11.1, U3.1 (I1)
- new net DIO_SV: J2.5 (Pin_5), R15.2, R19.1
- new net SCON_ALM: J5.10 (Pin_10), R18.1
- new net SCON_CSTP: J5.3 (Pin_3), U3.15 (O4)
- new net SCON_HEND: J5.9 (Pin_9), R17.1
- new net SCON_HOME: J5.4 (Pin_4), U3.16 (O3)
- new net SCON_INP: J5.8 (Pin_8), R16.1
- new net SCON_RES: J5.5 (Pin_5), U3.17 (O2)
- new net SCON_SON: J5.6 (Pin_6), U3.18 (O1)
- new net SCON_SV: J5.7 (Pin_7), R15.1
- new net VIN_REG: C5.1, D1.1 (K), U4.1 (Vin)
- no-connect marks 5 -> 9
Other:
- note added: "ALIMENTATION (une seule masse GND commune) J1 : 24 V de l'alimentation stabilisée externe. D1 : protection contre l'inversion de polarité. PS1 : régulateur à découpage 24 V -> 5 V, 1 A, SIP-3 (brochage 7805 : 1 = VIN, 2 = GND, 3 = VOUT). Le +24V alimente aussi U3 et le PIO du SCON."
- note added: "COMMANDES ADwin -> SCON (entrées PNP) U3 : drivers « source » 24 V. DIO haut = sortie U3 à +24 V. R11-R14 : SCON non commandé tant que le DIO-32 n'est pas initialisé. IN5-IN8 inutilisées reliées à GND."
- note added: "Depuis SCON-CB, sortie feedback (vérifier le brochage dans le manuel IAI) : Câble blindé, une paire torsadée par phase. Blindage à la terre d'un seul côté."
- note added: "J1 -> ADwin DIO-32 (TTL) 1-2 : sorties PULSE, SIGN 3-6 : sorties SON, RES, HOME, CSTP 7-10 : entrées SV, INP, HEND, ALM 11 : GND"
- note added: "J6 <-> SCON bornier PIO (PNP 24 V, mode impulsions) 1 = +24 V vers P24 (1A/2A) 2 = 0 V vers N (19B/20B) 3 = SON (5A) 4 = RES (6A) 5 = HOME (7A) 6 = CSTP (9A) 7 = SV 8 = INP (3B) 9 = HEND (4B) 10 = *ALM Broches SCON à vérifier dans le manuel ME0340."
- note added: "VERSION NON ISOLÉE : GND ADwin, 0 V du 24 V et masse des signaux SCON sont reliés. Relier les masses en un seul point au niveau de l'installation, câbles blindés, blindage d'un seul côté. Concrètement : Câbles entre la carte d'interface et le SCON (PULSE, feedback, PIO) : raccorder le blindage côté SCON, à la barre de terre de l'armoire ou à la borne de terre (FG/PE) du contrôleur. Côté carte, co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"
- note added: "ÉTATS SCON -> ADwin (sorties PNP 24 V) Diviseurs 10k / 2,2k : 24 V -> 4,3 V (26,4 V -> 4,8 V). Sortie SCON inactive : DIO tiré à 0 V par la 2,2k. *ALM actif à l'état bas (ON = pas d'alarme)."
- note removed: "C1 céramique au plus près de U1 (broche 16). C2 à l'arrivée du 5 V sur la carte."
- note removed: "Depuis SCON-CB, sortie feedback (vérifier le brochage dans le manuel IAI) : 1 = AFB 2 = /AFB 3 = BFB 4 = /BFB 5 = ZFB 6 = /ZFB 7 = masse signal (0 V de référence) Câble blindé, une paire torsadée par phase. Blindage à la terre d'un seul côté."
- note removed: "Une seule alimentation 5 V (J2) pour U1 et U2. U1/U2 montés sur supports DIP-16. AM26LS31CN / AM26LS32ACN compatibles broche à broche avec AM26C31 / AM26C32."
- note removed: "Vers ADwin (module compteur CO4-T, entrées TTL, brochage D-SUB à reporter) : 1 = A 2 = B 3 = Z (top zéro) 4 = masse (0 V commun ADwin)"
- note removed: "Vers ADwin DIO-32 : 1 = sortie TTL PULSE 2 = sortie TTL SIGN 3 = masse DIO (0 V commun)"
- moved on the sheet: C1, C3, R1, R10, R2, R3, R4, R5, R6, R7, R8, R9

Commit message: Modify BOM
Parts:
- C5: footprint Capacitor_THT:C_Disc_D5.0mm_W2.5mm_P5.00mm -> Capacitor_THT:C_Radial_D5.0mm_H11.0mm_P2.00mm
Changed lines of the file:
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@@
 			)
 		)
-		(property "Footprint" "Capacitor_THT:C_Disc_D5.0mm_W2.5mm_P5.00mm"
+		(property "Footprint" "Capacitor_THT:C_Radial_D5.0mm_H11.0mm_P2.00mm"
 			(at 73.66 27.94 0)
 			(hide yes)

Commit message: Add DEL Alim.
Parts:
- added D2, D3: WP710A10LGD, LED_THT:LED_D3.0mm, symbol Device:LED
- added R23: 10k, Resistor_THT:R_Axial_DIN0207_L6.3mm_D2.5mm_P7.62mm_Horizontal, symbol Device:R
- added R24: 2.2k, Resistor_THT:R_Axial_DIN0207_L6.3mm_D2.5mm_P7.62mm_Horizontal, symbol Device:R
- renumbered C6 to C2
Connections:
- net +24V: now also R23.1
- net +5V: now also R24.1
- net GND: now also D2.1 (K), D3.1 (K)
- new net: D3.2 (A), R24.2
- new net: D2.2 (A), R23.2

Commit message: Update Doc. and Gerber files
Parts:
- removed H1, H2, H3, H4: MountingHole, MountingHole:MountingHole_2.2mm_M2, symbol Mechanical:MountingHole

Commit message: Remove Hammond box, refactor schematic
Other:
- note added: "PARTIE PIO - Commandes servo - Lecture état servo SCON-CB entrées 24V commandées par TTL : SON, RES, HOM, CSTP SCON-CB sorties 24V adpatée en TTL SV, INP, HEN, ALM"
- note added: "Vers SCON-CB, connecteur PULSE 1 = PP (impulsion +) 2 = /PP (impulsion -) 3 = NP (sens +) 4 = /NP (sens -) Câble paires torsadées blindé : PP//PP dans une paire, NP//NP dans l'autre. Blindage à la terre d'un seul côté. Pas de 120 ohms côté SCON."
- note removed: "Alimentation 5 V régulée (4,75 à 5,25 V)"
- note removed: "C3 céramique au plus près de U2 (broche 16)."
- note removed: "Depuis SCON-CB, sortie feedback (vérifier le brochage dans le manuel IAI) : Câble blindé, une paire torsadée par phase. Blindage à la terre d'un seul côté."
- note removed: "G = +5 V et /G = 0 V : récepteurs toujours validés. Voie 4 inutilisée : 4A au +5 V, 4B à la masse (état défini, sortie 4Y non connectée)."
- note removed: "G = +5 V et /G = 0 V : sorties toujours validées. Entrées 3A et 4A inutilisées reliées à la masse (entrées CMOS jamais flottantes)."
- note removed: "J1 -> ADwin DIO-32 (TTL) 1-2 : sorties PULSE, SIGN 3-6 : sorties SON, RES, HOME, CSTP 7-10 : entrées SV, INP, HEND, ALM 11 : GND"
- note removed: "J6 <-> SCON bornier PIO (PNP 24 V, mode impulsions) 1 = +24 V vers P24 (1A/2A) 2 = 0 V vers N (19B/20B) 3 = SON (5A) 4 = RES (6A) 5 = HOME (7A) 6 = CSTP (9A) 7 = SV 8 = INP (3B) 9 = HEND (4B) 10 = *ALM Broches SCON à vérifier dans le manuel ME0340."
- note removed: "Vers SCON-CB, connecteur PULSE (vérifier le brochage dans le manuel IAI) : 1 = PP (impulsion +) 2 = /PP (impulsion -) 3 = NP (sens +) 4 = /NP (sens -) Câble paires torsadées blindé : PP//PP dans une paire, NP//NP dans l'autre. Blindage à la terre d'un seul côté. Pas de 120 ohms côté SCON sans recommandation du manuel."
- moved on the sheet: C1, C2, C3, C4, C5, D1, D2, D3, J1, J2, J3, J4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

Commit message: Update Doc.
Parts:
- added F1: Polyfuse, MF-R050:MFR050, symbol Device:Polyfuse
- added H1, H2, H3, H4, H5, H6: MountingHole, MountingHole:MountingHole_3.2mm_M3, symbol Mechanical:MountingHole
- added R25, R26, R28, R30: 10k, Resistor_THT:R_Axial_DIN0207_L6.3mm_D2.5mm_P7.62mm_Horizontal, symbol Device:R
- added R27, R29: 2.2k, Resistor_THT:R_Axial_DIN0207_L6.3mm_D2.5mm_P7.62mm_Horizontal, symbol Device:R
- C5: footprint Capacitor_THT:C_Radial_D5.0mm_H11.0mm_P2.00mm -> Capacitor_THT:CP_Radial_D5.0mm_P2.00mm; symbol Device:C -> Device:C_Polarized
- J2: value ADWIN_DIO32 -> Screw_Terminal_01x15; footprint TerminalBlock_Phoenix:TerminalBlock_Phoenix_MKDS-1,5-11-5.08_1x11_P5.08mm_Horizontal -> TerminalBlock_Phoenix:TerminalBlock_Phoenix_MKDS-1,5-15-5.08_1x15_P5.08mm_Horizontal; symbol Connector:Screw_Terminal_01x11 -> Connector:Screw_Terminal_01x15
- J5: value SCON_PIO -> Screw_Terminal_01x14; footprint TerminalBlock_Phoenix:TerminalBlock_Phoenix_MKDS-1,5-10-5.08_1x10_P5.08mm_Horizontal -> TerminalBlock_Phoenix:TerminalBlock_Phoenix_MKDS-1,5-14-5.08_1x14_P5.08mm_Horizontal; symbol Connector:Screw_Terminal_01x10 -> Connector:Screw_Terminal_01x14
Connections:
- net VIN_REG is gone; now on net +24V: C5.1, D1.1 (K), U4.1 (Vin)
- net +24V: no longer D1.2 (A), J1.1 (Pin_1)
- net DIO_CSTP: now also J2.11 (Pin_11); no longer J2.9 (Pin_9)
- net DIO_HOME: now also J2.10 (Pin_10); no longer J2.8 (Pin_8)
- net DIO_RES: now also J2.9 (Pin_9); no longer J2.7 (Pin_7)
- net DIO_SON: now also J2.8 (Pin_8); no longer J2.6 (Pin_6)
- net GND: now also R25.2, R26.2, R27.2, R29.2; no longer U3.5 (I5), U3.6 (I6)
- net SCON_ALM: now also J5.14 (Pin_14); no longer J5.10 (Pin_10)
- net SCON_CSTP: now also J5.5 (Pin_5); no longer J5.3 (Pin_3)
- net SCON_HEND: now also J5.13 (Pin_13); no longer J5.9 (Pin_9)
- net SCON_HOME: now also J5.6 (Pin_6); no longer J5.4 (Pin_4)
- net SCON_INP: now also J5.12 (Pin_12); no longer J5.8 (Pin_8)
- net SCON_RES: now also J5.7 (Pin_7); no longer J5.5 (Pin_5)
- net SCON_SON: now also J5.8 (Pin_8); no longer J5.6 (Pin_6)
- net SCON_SV: now also J5.11 (Pin_11); no longer J5.7 (Pin_7)
- net SCON_IN1: now reaches U3.13 (O6)
- net SCON_IN1: now also J5.3 (Pin_3)
- net SCON_IN0: now reaches U3.14 (O5)
- net SCON_IN0: now also J5.4 (Pin_4)
- net DIO_PULSE renamed DIO_PP
- net DIO_PP: now also J2.15 (Pin_15); no longer J2.11 (Pin_11)
- net DIO_SIGN renamed DIO_NP
- net DIO_NP: now also J2.14 (Pin_14); no longer J2.10 (Pin_10)
- net PULSE_N renamed PP_N
- net PULSE_P renamed PP_P
- net PULSE_TTL renamed PP_TTL
- net SIGN_N renamed NP_N
- net SIGN_P renamed NP_P
- net SIGN_TTL renamed NP_TTL
- new net: D1.2 (A), F1.2
- new net: F1.1, J1.1 (Pin_1)
- new net DIO_IN0: J2.6 (Pin_6), R27.1, R28.2
- new net DIO_IN1: J2.7 (Pin_7), R29.1, R30.2
- new net DIO_OUT0: J2.12 (Pin_12), R25.1, U3.5 (I5)
- new net DIO_OUT1: J2.13 (Pin_13), R26.1, U3.6 (I6)
- new net SCON_OUT0: J5.10 (Pin_10), R28.1
- new net SCON_OUT1: J5.9 (Pin_9), R30.1
- no-connect marks 9 -> 7
Other:
- note added: "Vers SCON-CB, connecteur PULSE 1 = PP 2 = /PP 3 = NP 4 = /NP Câble paires torsadées blindé : PP//PP dans une paire, NP//NP dans l'autre. Blindage à la terre d'un seul côté. Pas de 120 ohms côté SCON."
- note removed: "Vers SCON-CB, connecteur PULSE 1 = PP (impulsion +) 2 = /PP (impulsion -) 3 = NP (sens +) 4 = /NP (sens -) Câble paires torsadées blindé : PP//PP dans une paire, NP//NP dans l'autre. Blindage à la terre d'un seul côté. Pas de 120 ohms côté SCON."
- moved on the sheet: C2, D1, R11, R12, R13, R14, R15, R16, R17, R18, R19, R20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

Commit message: Update doc. Change PCB (RSTR, REND, *EMGS)
Connections:
- net DIO_IN0 renamed DIO_REN
- net DIO_IN1 renamed DIO_EMGS
- net DIO_OUT0 renamed RSTR
- net DIO_OUT1 renamed DIO_OUT
- net SCON_IN0 renamed SCON_RSTR
- net SCON_IN1 renamed SCON_IN
- net SCON_OUT0 renamed SCON_REN
- net SCON_OUT1 renamed SCON_EMGS
Changed lines of the file:
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@@
 		)
 	)
-	(label "DIO_IN1"
+	(label "DIO_EMGS"
 		(at 144.78 204.47 180)
 		(effects
@@
 		)
 	)
-	(label "SCON_IN0"
+	(label "SCON_RSTR"
 		(at 101.6 181.61 0)
 		(effects
@@
 		)
 	)
-	(label "SCON_IN0"
+	(label "SCON_RSTR"
 		(at 181.61 175.26 180)
 		(effects
@@
 		)
 	)
-	(label "DIO_OUT1"
+	(label "DIO_OUT"
 		(at 35.56 148.59 180)
 		(effects
@@
 		)
 	)
-	(label "DIO_OUT0"
+	(label "RSTR"
 		(at 31.75 93.98 0)
 		(effects
@@
 		)
 	)
-	(label "DIO_IN1"
+	(label "DIO_EMGS"
 		(at 31.75 106.68 0)
 		(effects
@@
 		)
 	)
-	(label "SCON_OUT1"
+	(label "SCON_EMGS"
 		(at 181.61 187.96 180)
 		(effects
@@
 		)
 	)
-	(label "DIO_OUT0"
+	(label "RSTR"
 		(at 81.28 181.61 180)
 		(effects
@@
 		)
 	)
-	(label "DIO_OUT1"
+	(label "DIO_OUT"
 		(at 81.28 184.15 180)
 		(effects
@@
 		)
 	)
-	(label "SCON_IN1"
+	(label "SCON_IN"
 		(at 101.6 184.15 0)
 		(effects
@@
 		)
 	)
-	(label "DIO_OUT1"
+	(label "DIO_OUT"
 		(at 31.75 91.44 0)
 		(effects
@@
 		)
 	)
-	(label "SCON_OUT0"
+	(label "SCON_REN"
 		(at 181.61 190.5 180)
 		(effects
@@
 		)
 	)
-	(label "SCON_IN1"
+	(label "SCON_IN"
 		(at 181.61 172.72 180)
 		(effects
@@
 		)
 	)
-	(label "DIO_OUT0"
+	(label "RSTR"
 		(at 25.4 148.59 180)
 		(effects
@@
 		)
 	)
-	(label "SCON_OUT1"
+	(label "SCON_EMGS"
 		(at 152.4 204.47 0)
 		(effects
@@
 		)
 	)
-	(label "SCON_OUT0"
+	(label "SCON_REN"
 		(at 124.46 204.47 0)
 		(effects
@@
 		)
 	)
-	(label "DIO_IN0"
+	(label "DIO_REN"
 		(at 116.84 204.47 180)
 		(effects
@@
 		)
 	)
-	(label "DIO_IN0"
+	(label "DIO_REN"
 		(at 31.75 109.22 0)
 		(effects
